Commit message: Complete integration of Panda arm and Trailer robot simulation stacks with warehouse_orchestrator

File: src/diff_robot/urdf/robot_remorque.urdf (robot description, URDF)
Before this commit: robot robot_remorque, 12 links, 11 joints
Links:
- added link trailer_cart_drop_point
Joints:
- added joint trailer_cart_drop_joint: type fixed, parent trailer_base_link, child trailer_cart_drop_point, origin xyz=0.4 0 0.15 rpy=0 0 0

File: src/diff_robot/urdf/tractor_ros2_control.xacro (robot description, xacro)
@@ -61,5 +61,5 @@
     <plugin filename="ign_ros2_control-system"
             name="ign_ros2_control::IgnitionROS2ControlPlugin">
-      <parameters>/home/rabeb/ros2_diff_drive_robot/src/diff_robot/config/diff_drive_controller.yaml</parameters>
+      <parameters>$(find diff_robot)/config/diff_drive_controller.yaml</parameters>
       <ros>
         <namespace>/</namespace>
